File: OverClock Hardware/Power_Supply.sch (KiCad schematic (older format))
At the start: 29 parts, among them J1 USB_C_Plug, U1 TLV62569, U2 AP7365, U3 10M02SCE144

Commit message: Place and route Decoupling Capacitors
Placed and routed all the decoupling capacitors for the FPGA. Created Top and bottom GND planes too for better signal integrity
Parts:
- C10, C11, C12, C13, C14, C15, C16, C17, C18, C19, C20, C21, C22, C6, C7, C8, C9: footprint Capacitor_SMD:C_0805_2012Metric_Pad1.15x1.40mm_HandSolder -> Capacitor_SMD:C_0603_1608Metric_Pad1.05x0.95mm_HandSolder
Changed lines of the file:
@@
 F 0 "C6" H 3992 5646 50  0000 L CNN
 F 1 "10nF" H 3992 5555 50  0000 L CNN
-F 2 "Capacitor_SMD:C_0805_2012Metric_Pad1.15x1.40mm_HandSolder" H 3900 5600 50  0001 C CNN
+F 2 "Capacitor_SMD:C_0603_1608Metric_Pad1.05x0.95mm_HandSolder" H 3900 5600 50  0001 C CNN
 F 3 "~" H 3900 5600 50  0001 C CNN
 	1    3900 5600
@@
 F 0 "C7" H 4342 5646 50  0000 L CNN
 F 1 "10nF" H 4342 5555 50  0000 L CNN
-F 2 "Capacitor_SMD:C_0805_2012Metric_Pad1.15x1.40mm_HandSolder" H 4250 5600 50  0001 C CNN
+F 2 "Capacitor_SMD:C_0603_1608Metric_Pad1.05x0.95mm_HandSolder" H 4250 5600 50  0001 C CNN
 F 3 "~" H 4250 5600 50  0001 C CNN
 	1    4250 5600
@@
 F 0 "C8" H 4692 5646 50  0000 L CNN
 F 1 "10nF" H 4692 5555 50  0000 L CNN
-F 2 "Capacitor_SMD:C_0805_2012Metric_Pad1.15x1.40mm_HandSolder" H 4600 5600 50  0001 C CNN
+F 2 "Capacitor_SMD:C_0603_1608Metric_Pad1.05x0.95mm_HandSolder" H 4600 5600 50  0001 C CNN
 F 3 "~" H 4600 5600 50  0001 C CNN
 	1    4600 5600
@@
 F 0 "C9" H 5042 5646 50  0000 L CNN
 F 1 "10nF" H 5042 5555 50  0000 L CNN
-F 2 "Capacitor_SMD:C_0805_2012Metric_Pad1.15x1.40mm_HandSolder" H 4950 5600 50  0001 C CNN
+F 2 "Capacitor_SMD:C_0603_1608Metric_Pad1.05x0.95mm_HandSolder" H 4950 5600 50  0001 C CNN
 F 3 "~" H 4950 5600 50  0001 C CNN
 	1    4950 5600
@@
 F 0 "C10" H 5392 5646 50  0000 L CNN
 F 1 "10nF" H 5392 5555 50  0000 L CNN
-F 2 "Capacitor_SMD:C_0805_2012Metric_Pad1.15x1.40mm_HandSolder" H 5300 5600 50  0001 C CNN
+F 2 "Capacitor_SMD:C_0603_1608Metric_Pad1.05x0.95mm_HandSolder" H 5300 5600 50  0001 C CNN
 F 3 "~" H 5300 5600 50  0001 C CNN
 	1    5300 5600
@@
 F 0 "C11" H 5742 5646 50  0000 L CNN
 F 1 "10nF" H 5742 5555 50  0000 L CNN
-F 2 "Capacitor_SMD:C_0805_2012Metric_Pad1.15x1.40mm_HandSolder" H 5650 5600 50  0001 C CNN
+F 2 "Capacitor_SMD:C_0603_1608Metric_Pad1.05x0.95mm_HandSolder" H 5650 5600 50  0001 C CNN
 F 3 "~" H 5650 5600 50  0001 C CNN
 	1    5650 5600
@@
 F 0 "C12" H 6092 5646 50  0000 L CNN
 F 1 "10nF" H 6092 5555 50  0000 L CNN
-F 2 "Capacitor_SMD:C_0805_2012Metric_Pad1.15x1.40mm_HandSolder" H 6000 5600 50  0001 C CNN
+F 2 "Capacitor_SMD:C_0603_1608Metric_Pad1.05x0.95mm_HandSolder" H 6000 5600 50  0001 C CNN
 F 3 "~" H 6000 5600 50  0001 C CNN
 	1    6000 5600
@@
 F 0 "C13" H 6442 5646 50  0000 L CNN
 F 1 "10nF" H 6442 5555 50  0000 L CNN
-F 2 "Capacitor_SMD:C_0805_2012Metric_Pad1.15x1.40mm_HandSolder" H 6350 5600 50  0001 C CNN
+F 2 "Capacitor_SMD:C_0603_1608Metric_Pad1.05x0.95mm_HandSolder" H 6350 5600 50  0001 C CNN
 F 3 "~" H 6350 5600 50  0001 C CNN
 	1    6350 5600
@@
 F 0 "C14" H 6792 5646 50  0000 L CNN
 F 1 "10nF" H 6792 5555 50  0000 L CNN
-F 2 "Capacitor_SMD:C_0805_2012Metric_Pad1.15x1.40mm_HandSolder" H 6700 5600 50  0001 C CNN
+F 2 "Capacitor_SMD:C_0603_1608Metric_Pad1.05x0.95mm_HandSolder" H 6700 5600 50  0001 C CNN
 F 3 "~" H 6700 5600 50  0001 C CNN
 	1    6700 5600
@@
 F 0 "C15" H 7142 5646 50  0000 L CNN
 F 1 "10nF" H 7142 5555 50  0000 L CNN
-F 2 "Capacitor_SMD:C_0805_2012Metric_Pad1.15x1.40mm_HandSolder" H 7050 5600 50  0001 C CNN
+F 2 "Capacitor_SMD:C_0603_1608Metric_Pad1.05x0.95mm_HandSolder" H 7050 5600 50  0001 C CNN
 F 3 "~" H 7050 5600 50  0001 C CNN
 	1    7050 5600
@@
 F 0 "C16" H 7492 5646 50  0000 L CNN
 F 1 "10nF" H 7492 5555 50  0000 L CNN
-F 2 "Capacitor_SMD:C_0805_2012Metric_Pad1.15x1.40mm_HandSolder" H 7400 5600 50  0001 C CNN
+F 2 "Capacitor_SMD:C_0603_1608Metric_Pad1.05x0.95mm_HandSolder" H 7400 5600 50  0001 C CNN
 F 3 "~" H 7400 5600 50  0001 C CNN
 	1    7400 5600
@@
 F 0 "C17" H 7842 5646 50  0000 L CNN
 F 1 "10nF" H 7842 5555 50  0000 L CNN
-F 2 "Capacitor_SMD:C_0805_2012Metric_Pad1.15x1.40mm_HandSolder" H 7750 5600 50  0001 C CNN
+F 2 "Capacitor_SMD:C_0603_1608Metric_Pad1.05x0.95mm_HandSolder" H 7750 5600 50  0001 C CNN
 F 3 "~" H 7750 5600 50  0001 C CNN
 	1    7750 5600
@@
 F 0 "C18" H 8192 5646 50  0000 L CNN
 F 1 "10nF" H 8192 5555 50  0000 L CNN
-F 2 "Capacitor_SMD:C_0805_2012Metric_Pad1.15x1.40mm_HandSolder" H 8100 5600 50  0001 C CNN
+F 2 "Capacitor_SMD:C_0603_1608Metric_Pad1.05x0.95mm_HandSolder" H 8100 5600 50  0001 C CNN
 F 3 "~" H 8100 5600 50  0001 C CNN
 	1    8100 5600
@@
 F 0 "C19" H 8542 5646 50  0000 L CNN
 F 1 "10nF" H 8542 5555 50  0000 L CNN
-F 2 "Capacitor_SMD:C_0805_2012Metric_Pad1.15x1.40mm_HandSolder" H 8450 5600 50  0001 C CNN
+F 2 "Capacitor_SMD:C_0603_1608Metric_Pad1.05x0.95mm_HandSolder" H 8450 5600 50  0001 C CNN
 F 3 "~" H 8450 5600 50  0001 C CNN
 	1    8450 5600
@@
 F 0 "C20" H 8892 5646 50  0000 L CNN
 F 1 "10nF" H 8892 5555 50  0000 L CNN
-F 2 "Capacitor_SMD:C_0805_2012Metric_Pad1.15x1.40mm_HandSolder" H 8800 5600 50  0001 C CNN
+F 2 "Capacitor_SMD:C_0603_1608Metric_Pad1.05x0.95mm_HandSolder" H 8800 5600 50  0001 C CNN
 F 3 "~" H 8800 5600 50  0001 C CNN
 	1    8800 5600
@@
 F 0 "C21" H 9242 5646 50  0000 L CNN
 F 1 "10nF" H 9242 5555 50  0000 L CNN
-F 2 "Capacitor_SMD:C_0805_2012Metric_Pad1.15x1.40mm_HandSolder" H 9150 5600 50  0001 C CNN
+F 2 "Capacitor_SMD:C_0603_1608Metric_Pad1.05x0.95mm_HandSolder" H 9150 5600 50  0001 C CNN
 F 3 "~" H 9150 5600 50  0001 C CNN
 	1    9150 5600
@@
 F 0 "C22" H 9592 5646 50  0000 L CNN
 F 1 "10nF" H 9592 5555 50  0000 L CNN
-F 2 "Capacitor_SMD:C_0805_2012Metric_Pad1.15x1.40mm_HandSolder" H 9500 5600 50  0001 C CNN
+F 2 "Capacitor_SMD:C_0603_1608Metric_Pad1.05x0.95mm_HandSolder" H 9500 5600 50  0001 C CNN
 F 3 "~" H 9500 5600 50  0001 C CNN
 	1    9500 5600
@@
 One Decoupling Cap per Vcc Pin.\nPlace physically as close to pin as possible
 $Comp
-L power:PWR_FLAG #FLG0101
+L power:PWR_FLAG #FLG01
 U 1 1 5CBC6DC8
 P 2800 1400
-F 0 "#FLG0101" H 2800 1475 50  0001 C CNN
+F 0 "#FLG01" H 2800 1475 50  0001 C CNN
 F 1 "PWR_FLAG" H 2800 1574 50  0000 C CNN
 F 2 "" H 2800 1400 50  0001 C CNN
@@
 	2800 1400 3350 1400
 $Comp
-L power:PWR_FLAG #FLG0102
+L power:PWR_FLAG #FLG04
 U 1 1 5CBC6E7D
 P 3350 2000
-F 0 "#FLG0102" H 3350 2075 50  0001 C CNN
+F 0 "#FLG04" H 3350 2075 50  0001 C CNN
 F 1 "PWR_FLAG" H 3350 2173 50  0000 C CNN
 F 2 "" H 3350 2000 50  0001 C CNN
@@
 Connection ~ 3350 2000
 $Comp
-L power:PWR_FLAG #FLG0103
+L power:PWR_FLAG #FLG03
 U 1 1 5CBC6F6A
 P 7250 1400
-F 0 "#FLG0103" H 7250 1475 50  0001 C CNN
+F 0 "#FLG03" H 7250 1475 50  0001 C CNN
 F 1 "PWR_FLAG" H 7250 1574 50  0000 C CNN
 F 2 "" H 7250 1400 50  0001 C CNN
@@
 	7250 1400 7400 1400
 $Comp
-L power:PWR_FLAG #FLG0104
+L power:PWR_FLAG #FLG02
 U 1 1 5CBC7C86
 P 6150 1400
-F 0 "#FLG0104" H 6150 1475 50  0001 C CNN
+F 0 "#FLG02" H 6150 1475 50  0001 C CNN
 F 1 "PWR_FLAG" H 6150 1574 50  0000 C CNN
 F 2 "" H 6150 1400 50  0001 C CNN
