File: OverClock Hardware/FPGA_Interfacing.sch (KiCad schematic (older format))
At the start: 20 parts, among them J2 JTAG_HDR, J3 Conn_01x03_Female, SW1 Switch_Momentary, SW2 Switch_Momentary, SW3 Switch_Momentary, SW4 Switch_Momentary, U3 10M02SCE144

Commit message: Completed Initial Routing
Parts:
- R3, R4, R5, R6: footprint Resistor_SMD:R_0805_2012Metric_Pad1.15x1.40mm_HandSolder -> Resistor_SMD:R_0603_1608Metric_Pad1.05x0.95mm_HandSolder
Connections:
- net H+: now also R7.2, SW1.1, SW1.3, U3.130 (GPIO_8_16/CRC_Err); no longer R10.2, SW4.1, SW4.3, U3.127 (GPIO_8_13)
- net H-: now also R8.2, SW2.1, SW2.3, U3.129 (GPIO_8_15); no longer R9.2, SW3.1, SW3.3, U3.128 (GPIO_8_14)
- net M+: now also R9.2, SW3.1, SW3.3, U3.128 (GPIO_8_14); no longer R8.2, SW2.1, SW2.3, U3.129 (GPIO_8_15)
- net M-: now also R10.2, SW4.1, SW4.3, U3.127 (GPIO_8_13); no longer R7.2, SW1.1, SW1.3, U3.130 (GPIO_8_16/CRC_Err)
Changed lines of the file:
@@
 F 0 "R5" H 5559 2646 50  0000 L CNN
 F 1 "1K" H 5559 2555 50  0000 L CNN
-F 2 "Resistor_SMD:R_0805_2012Metric_Pad1.15x1.40mm_HandSolder" H 5500 2600 50  0001 C CNN
+F 2 "Resistor_SMD:R_0603_1608Metric_Pad1.05x0.95mm_HandSolder" H 5500 2600 50  0001 C CNN
 F 3 "~" H 5500 2600 50  0001 C CNN
 	1    5500 2600
@@
 F 0 "R6" H 5809 2646 50  0000 L CNN
 F 1 "1K" H 5809 2555 50  0000 L CNN
-F 2 "Resistor_SMD:R_0805_2012Metric_Pad1.15x1.40mm_HandSolder" H 5750 2600 50  0001 C CNN
+F 2 "Resistor_SMD:R_0603_1608Metric_Pad1.05x0.95mm_HandSolder" H 5750 2600 50  0001 C CNN
 F 3 "~" H 5750 2600 50  0001 C CNN
 	1    5750 2600
@@
 F 0 "R3" H 5659 1746 50  0000 L CNN
 F 1 "1K" H 5659 1655 50  0000 L CNN
-F 2 "Resistor_SMD:R_0805_2012Metric_Pad1.15x1.40mm_HandSolder" H 5600 1700 50  0001 C CNN
+F 2 "Resistor_SMD:R_0603_1608Metric_Pad1.05x0.95mm_HandSolder" H 5600 1700 50  0001 C CNN
 F 3 "~" H 5600 1700 50  0001 C CNN
 	1    5600 1700
@@
 F 0 "R4" H 5959 1746 50  0000 L CNN
 F 1 "1K" H 5959 1655 50  0000 L CNN
-F 2 "Resistor_SMD:R_0805_2012Metric_Pad1.15x1.40mm_HandSolder" H 5900 1700 50  0001 C CNN
+F 2 "Resistor_SMD:R_0603_1608Metric_Pad1.05x0.95mm_HandSolder" H 5900 1700 50  0001 C CNN
 F 3 "~" H 5900 1700 50  0001 C CNN
 	1    5900 1700
@@
 Text Label 5200 2250 0    50   ~ 0
 TDO
+Text Label 5300 5650 2    50   ~ 0
+H+
+Text Label 5300 5550 2    50   ~ 0
+H-
+Text Label 5300 5450 2    50   ~ 0
+M+
 Text Label 5300 5350 2    50   ~ 0
-H+
-Text Label 5300 5450 2    50   ~ 0
-H-
-Text Label 5300 5550 2    50   ~ 0
-M+
-Text Label 5300 5650 2    50   ~ 0
 M-
 $Comp
